Commit message: added the flamingo config

File: resources/robots/flamingo/urdf/flamingo.urdf (robot description, URDF)
Before this commit: robot biped-wireframe-simplified-sat-urdf, 21 links, 20 joints
Links:
- link ankle-l_1: geometry collision mesh filename=../meshes/ankle-l_1.stl scale=0.001 0.001 0.001; visual mesh filename=../meshes/ankle-l_1.stl scale=0.001 0.001 0.001
- link ankle-r_1: geometry collision mesh filename=../meshes/ankle-r_1.stl scale=0.001 0.001 0.001; visual mesh filename=../meshes/ankle-r_1.stl scale=0.001 0.001 0.001
- link base_link: geometry collision mesh filename=../meshes/base_link.stl scale=0.001 0.001 0.001; visual mesh filename=../meshes/base_link.stl scale=0.001 0.001 0.001
- link foot-l_1: geometry collision mesh filename=../meshes/foot-l_1.stl scale=0.001 0.001 0.001; visual mesh filename=../meshes/foot-l_1.stl scale=0.001 0.001 0.001
- link foot-r_1: geometry collision mesh filename=../meshes/foot-r_1.stl scale=0.001 0.001 0.001; visual mesh filename=../meshes/foot-r_1.stl scale=0.001 0.001 0.001
- link hip-link-l_1: geometry collision mesh filename=../meshes/hip-link-l_1.stl scale=0.001 0.001 0.001; visual mesh filename=../meshes/hip-link-l_1.stl scale=0.001 0.001 0.001
- link hip-link-r_1: geometry collision mesh filename=../meshes/hip-link-r_1.stl scale=0.001 0.001 0.001; visual mesh filename=../meshes/hip-link-r_1.stl scale=0.001 0.001 0.001
- link hip-pitch-l_1: geometry collision mesh filename=../meshes/hip-pitch-l_1.stl scale=0.001 0.001 0.001; visual mesh filename=../meshes/hip-pitch-l_1.stl scale=0.001 0.001 0.001
- link hip-pitch-r_1: geometry collision mesh filename=../meshes/hip-pitch-r_1.stl scale=0.001 0.001 0.001; visual mesh filename=../meshes/hip-pitch-r_1.stl scale=0.001 0.001 0.001
- link hip-roll-l_1: geometry collision mesh filename=../meshes/hip-roll-l_1.stl scale=0.001 0.001 0.001; visual mesh filename=../meshes/hip-roll-l_1.stl scale=0.001 0.001 0.001
- link hip-roll-r_1: geometry collision mesh filename=../meshes/hip-roll-r_1.stl scale=0.001 0.001 0.001; visual mesh filename=../meshes/hip-roll-r_1.stl scale=0.001 0.001 0.001
- link knee-l_1: geometry collision mesh filename=../meshes/knee-l_1.stl scale=0.001 0.001 0.001; visual mesh filename=../meshes/knee-l_1.stl scale=0.001 0.001 0.001
- link knee-r_1: geometry collision mesh filename=../meshes/knee-r_1.stl scale=0.001 0.001 0.001; visual mesh filename=../meshes/knee-r_1.stl scale=0.001 0.001 0.001
- link tarsal-l_1: geometry collision mesh filename=../meshes/tarsal-l_1.stl scale=0.001 0.001 0.001; visual mesh filename=../meshes/tarsal-l_1.stl scale=0.001 0.001 0.001
- link tarsal-r_1: mass 0.07751176852113108 -> 0.07751176852113106; geometry collision mesh filename=../meshes/tarsal-r_1.stl scale=0.001 0.001 0.001; visual mesh filename=../meshes/tarsal-r_1.stl scale=0.001 0.001 0.001
- link thigh-l_1: geometry collision mesh filename=../meshes/thigh-l_1.stl scale=0.001 0.001 0.001; visual mesh filename=../meshes/thigh-l_1.stl scale=0.001 0.001 0.001
- link thigh-r_1: geometry collision mesh filename=../meshes/thigh-r_1.stl scale=0.001 0.001 0.001; visual mesh filename=../meshes/thigh-r_1.stl scale=0.001 0.001 0.001
- link tibia-l_1: geometry collision mesh filename=../meshes/tibia-l_1.stl scale=0.001 0.001 0.001; visual mesh filename=../meshes/tibia-l_1.stl scale=0.001 0.001 0.001
- link tibia-r_1: geometry collision mesh filename=../meshes/tibia-r_1.stl scale=0.001 0.001 0.001; visual mesh filename=../meshes/tibia-r_1.stl scale=0.001 0.001 0.001
- link toes-l_1: geometry collision mesh filename=../meshes/toes-l_1.stl scale=0.001 0.001 0.001; visual mesh filename=../meshes/toes-l_1.stl scale=0.001 0.001 0.001
- link toes-r_1: geometry collision mesh filename=../meshes/toes-r_1.stl scale=0.001 0.001 0.001; visual mesh filename=../meshes/toes-r_1.stl scale=0.001 0.001 0.001
Joints:
- removed joint Revolute 123
- removed joint Revolute 125
- removed joint Revolute 127
- removed joint Revolute 129
- removed joint Revolute 131
- removed joint Revolute 133
- removed joint Revolute 135
- removed joint Revolute 137
- removed joint Revolute 139
- removed joint Revolute 141
- removed joint Rigid 122
- removed joint Rigid 124
- removed joint Rigid 126
- removed joint Rigid 128
- removed joint Rigid 130
- removed joint Rigid 132
- removed joint Rigid 134
- removed joint Rigid 136
- removed joint Rigid 138
- removed joint Rigid 140
- added joint ankle_l: type continuous, parent ankle-l_1, child tarsal-l_1, origin xyz=0.0 0.0 0.0 rpy=0 0 0, axis 1.0 0.0 0.0
- added joint ankle_r: type continuous, parent ankle-r_1, child tarsal-r_1, origin xyz=0.0 0.0 0.0 rpy=0 0 0, axis 1.0 -0.0 0.0
- added joint feet_l: type continuous, parent toes-l_1, child foot-l_1, origin xyz=0.0 0.0 0.0 rpy=0 0 0, axis -1.0 0.0 0.0
- added joint feet_r: type continuous, parent toes-r_1, child foot-r_1, origin xyz=0.0 0.0 0.0 rpy=0 0 0, axis -1.0 -0.0 -0.0
- added joint fixed_ankle_l: type fixed, parent tibia-l_1, child ankle-l_1, origin xyz=0.0 0.12 -0.207846 rpy=0 0 0
- added joint fixed_ankle_r: type fixed, parent tibia-r_1, child ankle-r_1, origin xyz=0.0 0.12 -0.207846 rpy=0 0 0
- added joint fixed_hip_pitch_l: type fixed, parent hip-link-l_1, child hip-pitch-l_1, origin xyz=0.0 0.092 0.0 rpy=0 0 0
- added joint fixed_hip_pitch_r: type fixed, parent hip-link-r_1, child hip-pitch-r_1, origin xyz=0.0 0.092 0.0 rpy=0 0 0
- added joint fixed_hip_roll_l: type fixed, parent base_link, child hip-roll-l_1, origin xyz=0.08 0.0 0.0 rpy=0 0 0
- added joint fixed_hip_roll_r: type fixed, parent base_link, child hip-roll-r_1, origin xyz=-0.08 0.008 0.0 rpy=0 0 0
- added joint fixed_knee_l: type fixed, parent thigh-l_1, child knee-l_1, origin xyz=0.0 -0.075 -0.129904 rpy=0 0 0
- added joint fixed_knee_r: type fixed, parent thigh-r_1, child knee-r_1, origin xyz=0.0 -0.075 -0.129904 rpy=0 0 0
- added joint fixed_toe_l: type fixed, parent tarsal-l_1, child toes-l_1, origin xyz=0.0 -0.190526 -0.11 rpy=0 0 0
- added joint fixed_toe_r: type fixed, parent tarsal-r_1, child toes-r_1, origin xyz=0.0 -0.190526 -0.11 rpy=0 0 0
- added joint hip_pitch_l: type continuous, parent hip-pitch-l_1, child thigh-l_1, origin xyz=0.0 0.0 0.0 rpy=0 0 0, axis -1.0 0.0 0.0
- added joint hip_pitch_r: type continuous, parent hip-pitch-r_1, child thigh-r_1, origin xyz=0.0 0.0 0.0 rpy=0 0 0, axis -1.0 -0.0 0.0
- added joint hip_roll_l: type continuous, parent hip-roll-l_1, child hip-link-l_1, origin xyz=0.0 0.0205 -0.0 rpy=0 0 0, axis 0.0 1.0 -0.0
- added joint hip_roll_r: type continuous, parent hip-roll-r_1, child hip-link-r_1, origin xyz=0.0 0.0205 0.0 rpy=0 0 0, axis 0.0 1.0 -0.0
- added joint knee_l: type continuous, parent knee-l_1, child tibia-l_1, origin xyz=0.0 0.0 0.0 rpy=0 0 0, axis -1.0 -0.0 -0.0
- added joint knee_r: type continuous, parent knee-r_1, child tibia-r_1, origin xyz=0.0 0.0 0.0 rpy=0 0 0, axis -1.0 0.0 -0.0

Commit message: fixed pid values

File: resources/robots/flamingo/urdf/flamingo.urdf (robot description, URDF)
Before this commit: robot biped-wireframe-simplified-sat-urdf, 21 links, 20 joints
Joints:
- joint ankle_l: type continuous -> revolute
- joint ankle_r: type continuous -> revolute
- joint feet_l: type continuous -> revolute
- joint feet_r: type continuous -> revolute
- joint hip_pitch_l: type continuous -> revolute
- joint hip_pitch_r: type continuous -> revolute
- joint hip_roll_l: type continuous -> revolute
- joint hip_roll_r: type continuous -> revolute
- joint knee_l: type continuous -> revolute
- joint knee_r: type continuous -> revolute
